Commit message: added collision and inertia

File: description/robot_core.xacro (robot description, xacro)
@@ -10,4 +10,28 @@
     <xacro:property name="wheel_xoff" value="0.2" />
     <xacro:property name="caster_xoff" value="0.24" />
+    <!-- Define intertial property macros  -->
+    <xacro:macro name="box_inertia" params="m w h d">
+        <inertial>
+            <origin xyz="0 0 0" rpy="${pi/2} 0 ${pi/2}" />
+            <mass value="${m}" />
+            <inertia ixx="${(m/12) * (h*h + d*d)}" ixy="0.0" ixz="0.0" iyy="${(m/12) * (w*w + d*d)}"
+                iyz="0.0" izz="${(m/12) * (w*w + h*h)}" />
+        </inertial>
+    </xacro:macro>
+    <xacro:macro name="cylinder_inertia" params="m r h">
+        <inertial>
+            <origin xyz="0 0 0" rpy="${pi/2} 0 0" />
+            <mass value="${m}" />
+            <inertia ixx="${(m/12) * (3*r*r + h*h)}" ixy="0" ixz="0" iyy="${(m/12) * (3*r*r + h*h)}"
+                iyz="0" izz="${(m/2) * (r*r)}" />
+        </inertial>
+    </xacro:macro>
+    <xacro:macro name="sphere_inertia" params="m r">
+        <inertial>
+            <mass value="${m}" />
+            <inertia ixx="${(2/5) * m * (r*r)}" ixy="0.0" ixz="0.0" iyy="${(2/5) * m * (r*r)}"
+                iyz="0.0" izz="${(2/5) * m * (r*r)}" />
+        </inertial>
+    </xacro:macro>
     <!-- Robot Base -->
     <link name="base_link">
@@ -20,4 +44,10 @@
             </material>
         </visual>
+        <collision>
+            <geometry>
+                <box size="${base_length} ${base_width} ${base_height}" />
+            </geometry>
+        </collision>
+        <xacro:box_inertia m="15" w="${base_width}" d="${base_length}" h="${base_height}" />
     </link>
     <!-- Robot Footprint -->
@@ -40,4 +70,11 @@
                 </material>
             </visual>
+            <collision>
+                <origin xyz="0 0 0" rpy="${pi/2} 0 0" />
+                <geometry>
+                    <cylinder radius="${wheel_radius}" length="${wheel_width}" />
+                </geometry>
+            </collision>
+            <xacro:cylinder_inertia m="0.5" r="${wheel_radius}" h="${wheel_width}" />
         </link>
         <joint name="${prefix}_joint" type="continuous">
@@ -62,4 +99,11 @@
             </material>
         </visual>
+        <collision>
+            <origin xyz="0 0 0" rpy="0 0 0" />
+            <geometry>
+                <sphere radius="${(wheel_radius+wheel_zoff-(base_height/2))}" />
+            </geometry>
+        </collision>
+        <xacro:sphere_inertia m="0.5" r="${(wheel_radius+wheel_zoff-(base_height/2))}" />
     </link>
     <joint name="caster_r_joint" type="fixed">
@@ -77,4 +121,11 @@
             </material>
         </visual>
+        <collision>
+            <origin xyz="0 0 0" rpy="0 0 0" />
+            <geometry>
+                <sphere radius="${(wheel_radius+wheel_zoff-(base_height/2))}" />
+            </geometry>
+        </collision>
+        <xacro:sphere_inertia m="0.5" r="${(wheel_radius+wheel_zoff-(base_height/2))}" />
     </link>
     <joint name="caster_l_joint" type="fixed">

Commit message: added gazebo tags as well as control

File: description/robot_core.xacro (robot description, xacro)
@@ -78,4 +78,7 @@
             <xacro:cylinder_inertia m="0.5" r="${wheel_radius}" h="${wheel_width}" />
         </link>
+        <gazebo reference="${prefix}_link">
+            <material>Gazebo/Black</material>
+        </gazebo>
         <joint name="${prefix}_joint" type="continuous">
             <parent link="base_link" />
@@ -107,4 +110,9 @@
         <xacro:sphere_inertia m="0.5" r="${(wheel_radius+wheel_zoff-(base_height/2))}" />
     </link>
+    <gazebo reference="front_r_caster">
+        <material>Gazebo/Black</material>
+        <mu1 value="0.001"/>
+        <mu2 value="0.001"/>
+    </gazebo>
     <joint name="caster_r_joint" type="fixed">
         <parent link="base_link" />
@@ -129,4 +137,9 @@
         <xacro:sphere_inertia m="0.5" r="${(wheel_radius+wheel_zoff-(base_height/2))}" />
     </link>
+    <gazebo reference="front_l_caster">
+        <material>Gazebo/Black</material>
+        <mu1 value="0.001"/>
+        <mu2 value="0.001"/>
+    </gazebo>
     <joint name="caster_l_joint" type="fixed">
         <parent link="base_link" />
